File: CVinoutAxov2.sch (KiCad schematic (older format))
At the start: 75 parts, among them J1 CVin A, J10 audio_in L, J11 audio_in R, J12 Conn_01x04, J13 audio_out L, J14 audio_out R, J15 USB_A, J16 Conn_01x04, J17 Conn_01x02, J2 CVin B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

Commit message: added disc caps
Parts:
- C3, C4, C5, C6: footprint Capacitor_THT:C_Disc_D12.5mm_W5.0mm_P7.50mm -> Capacitor_THT:C_Disc_D5.0mm_W2.5mm_P2.50mm
Changed lines of the file:
@@
 F 0 "C6" V 5671 1450 50  0000 C CNN
 F 1 "C_Small" V 5762 1450 50  0000 C CNN
-F 2 "Capacitor_THT:C_Disc_D12.5mm_W5.0mm_P7.50mm" H 5900 1450 50  0001 C CNN
+F 2 "Capacitor_THT:C_Disc_D5.0mm_W2.5mm_P2.50mm" H 5900 1450 50  0001 C CNN
 F 3 "~" H 5900 1450 50  0001 C CNN
 	1    5900 1450
@@
 F 0 "C5" V 5671 850 50  0000 C CNN
 F 1 "C_Small" V 5762 850 50  0000 C CNN
-F 2 "Capacitor_THT:C_Disc_D12.5mm_W5.0mm_P7.50mm" H 5900 850 50  0001 C CNN
+F 2 "Capacitor_THT:C_Disc_D5.0mm_W2.5mm_P2.50mm" H 5900 850 50  0001 C CNN
 F 3 "~" H 5900 850 50  0001 C CNN
 	1    5900 850
@@
 F 0 "C4" V 2371 1050 50  0000 C CNN
 F 1 "C_Small" V 2462 1050 50  0000 C CNN
-F 2 "Capacitor_THT:C_Disc_D12.5mm_W5.0mm_P7.50mm" H 2600 1050 50  0001 C CNN
+F 2 "Capacitor_THT:C_Disc_D5.0mm_W2.5mm_P2.50mm" H 2600 1050 50  0001 C CNN
 F 3 "~" H 2600 1050 50  0001 C CNN
 	1    2600 1050
@@
 F 0 "C3" V 2271 1650 50  0000 C CNN
 F 1 "C_Small" V 2362 1650 50  0000 C CNN
-F 2 "Capacitor_THT:C_Disc_D12.5mm_W5.0mm_P7.50mm" H 2500 1650 50  0001 C CNN
+F 2 "Capacitor_THT:C_Disc_D5.0mm_W2.5mm_P2.50mm" H 2500 1650 50  0001 C CNN
 F 3 "~" H 2500 1650 50  0001 C CNN
 	1    2500 1650
